File: hardware/main.kicad_pcb (KiCad board)
At the start: 4 copper layers, 88 x 111 mm, 526 parts, among them J1 DS1128-09-S8B8X, J2 DS1128-09-S8B8X, J3 DS1128-09-S8B8X, J4 SMA-KWE901, J5 SMA-KWE901, J6 IDC-08M, J7 IDC-08M, J8 USB_C_Receptacle, J9 TYPE-C-31-M-12, Q1 SSM6J501NU, Q2 SSM6J501NU, Q3 FDV301N, Q4 BC817, SW1 TS-1187A-B-A-B, SW2 TS-1187A-B-A-B, SW3 TS-1187A-B-A-B, SW4 TS-1187A-B-A-B, U1 SN74LVC1G175, U10 W25Q256FVEIG, U11 MT7603E, U12 TPD2EUSB30, U13 TPD2EUSB30, U14 TPD2EUSB30, U15 IP5328P, U16 N096-2864KSWEG01-H30, U2 MT7621A, U3 TPS63020, U4 TPS63020, U5 MT3420B, U6 MT3420B, U7 MT3420B, U8 MT3420B, U9 NT5CB64M16FP-DH (!), X1 HSO321S-50MHZ-3.3V, Y1 X322540MPB4SI

Commit message: init pcb
Parts:
- removed BT1, BT2, BT3, BT4: BH-18650-B1BA002, MAS_Package_nostd:BatteryHolder_BH-18650-B1BA002
- removed C100, C101, C102, C104, C106, C109, C110, C137, C140, C143, C144, C146, C147, C148, C149, C150, C153, C154, C155, C156, C159, C160, C161, C162, C164, C165, C166, C167, C168, C169, C170, C171, C172, C173, C178, C183, C184, C185, C193, C194, C196, C197, C90, C91, C92, C93, C94, C95, C96, C97, C98, C99: 100n, Capacitor_SMD:C_0603_1608Metric
- removed C103, C142, C202, C203: 4.7u, Capacitor_SMD:C_0805_2012Metric
- removed C105, C107, C108: 1n, Capacitor_SMD:C_0805_2012Metric
- removed C115, C116: 9p, Capacitor_SMD:C_0603_1608Metric
- removed C117, C118, C119, C120: 1.2p, Capacitor_SMD:C_0603_1608Metric
- removed C121, C122, C123, C124: 10p, Capacitor_SMD:C_0603_1608Metric
- removed C125, C126, C127, C128: 0.5p, Capacitor_SMD:C_0603_1608Metric
- removed C129, C130, C131, C132: 3p, Capacitor_SMD:C_0603_1608Metric
- removed C133, C134, C135, C136, C139, C195, C198, C199, C200, C201: 1u, Capacitor_SMD:C_0603_1608Metric
- removed C138, C186, C189, C191: 22u, Capacitor_SMD:C_0805_2012Metric
- removed C141, C152, C158, C180, C187, C188, C190, C192: 10u, Capacitor_SMD:C_0805_2012Metric
- removed C151, C157, C181, C182: 2.2u, Capacitor_SMD:C_0805_2012Metric
- removed C163, C176, C177, C179: 470n, Capacitor_SMD:C_0603_1608Metric
- removed C174 (x2), C175 (x2): 18p, Capacitor_SMD:C_0603_1608Metric
- removed the C57 at (34.3, -70.5)
- removed the C57 at (143.7, -69.8)
- removed the C58 at (139.1, -60.3)
- removed the C58 at (29.6, -61.0)
- removed the C59 at (36.6, -63.6)
- removed the C59 at (146.1, -62.9)
- removed the C60 at (29.6, -64.1)
- removed the C60 at (139.1, -63.4)
- removed the C61 at (143.7, -60.3)
- removed the C61 at (34.3, -61.0)
- removed the C62 at (141.2, -69.8)
- removed the C62 at (31.8, -70.5)
- removed the C63 at (24.8, -67.3)
- removed the C63 at (134.2, -66.6)
- removed the C64 at (134.2, -69.8)
- removed the C64 at (24.8, -70.5)
- removed the C65 at (137.4, -60.3)
- removed the C65 at (27.9, -61.0)
- removed the C66 at (131.5, -66.1)
- removed the C66 at (22.1, -66.8)
- removed the C67 at (136.8, -69.8)
- removed the C67 at (27.3, -70.5)
- removed the C68 at (31.8, -67.3)
- removed the C68 at (141.2, -66.6)
- removed the C69 at (143.7, -66.6)
- removed the C69 at (34.3, -67.3)
- removed the C70 at (143.7, -63.4)
- removed the C70 at (34.3, -64.1)
- removed the C71 at (36.6, -60.6)
- removed the C71 at (146.1, -59.9)
- removed the C72 at (134.2, -60.3)
- removed the C72 at (24.8, -61.0)
- removed the C73 at (20.8, -53.8)
- removed the C73 at (130.3, -53.1)
- removed the C74 at (134.2, -63.4)
- removed the C74 at (24.8, -64.1)
- removed the C75 at (132.1, -71.7)
- removed the C75 at (22.6, -72.4)
- removed the C76 at (20.6, -72.4)
- removed the C76 at (130.0, -71.7)
- removed F2, F3, F4: 0466001.NRHF, MAS_Package_std:Fuse_1812_4532Metric
- removed J4, J5: SMA-KWE901, MAS_Package_std:SMA_Amphenol_901-143_Horizontal
- removed J6, J7: IDC-08M, Connector_PinHeader_1.27mm:PinHeader_2x04_P1.27mm_Vertical
- removed J8: USB_C_Receptacle, Connector_USB:USB_C_Receptacle_HRO_TYPE-C-31-M-12
- removed J9: TYPE-C-31-M-12, MAS_Package_std:USB_C_Receptacle_HRO_TYPE-C-31-M-12
- removed JP3, JP4, JP5, JP6, JP7: J_Boot, Jumper:SolderJumper-2_P1.3mm_Open_Pad1.0x1.5mm
- removed L11, L12: SDCL1608C1N2STDF, Inductor_SMD:L_0603_1608Metric
- removed L13, L14, L15, L16: HK16082N7S-T, Inductor_SMD:L_0603_1608Metric
- removed L17, L18, L19, L20: VHF160808H1N8ST, Inductor_SMD:L_0603_1608Metric
- removed L21, L22, L23, L24: SDCL1608C3N0STDF, Inductor_SMD:L_0603_1608Metric
- removed L25, L26: SLO0530H2R2MTT, MAS_Package_std:Power_inductor_SMD_0530
- removed L8: CBM160808U121T, Inductor_SMD:L_0603_1608Metric
- removed Q1, Q2: SSM6J501NU, MAS_Package_std:U-MOSVI
- removed Q3: FDV301N, Package_TO_SOT_SMD:SOT-23
- removed Q4: BC817, Package_TO_SOT_SMD:SOT-23
- removed the R10 at (36.6, -62.1)
- removed the R10 at (146.1, -61.4)
- removed R100 (x2), R103: 24k, Resistor_SMD:R_0603_1608Metric
- removed R101, R102: 22k, Resistor_SMD:R_0603_1608Metric
- removed R104, R105, R106, R107, R108, R113, R114, R161, R165, R168, R169, R170, R171, R72, R81, R86, R98, R99: 0R, Resistor_SMD:R_0603_1608Metric
- removed R109, R110, R111, R112: 51R, Resistor_SMD:R_0603_1608Metric
- removed the R11 at (146.1, -64.4)
- removed the R11 at (36.6, -65.1)
- removed R115, R125: 10k, Resistor_SMD:R_0603_1608Metric
- removed R116, R127, R90: 1k, Resistor_SMD:R_0603_1608Metric
- removed R117: 0.01R, Resistor_SMD:R_1206_3216Metric
- removed R118: 82k, Resistor_SMD:R_0603_1608Metric
- removed R119, R128: 100k, Resistor_SMD:R_0603_1608Metric
- removed R120: 100k (NTC), Resistor_SMD:R_0805_2012Metric
- removed R121, R130, R131, R134, R136, R137, R139, R141, R143, R146, R147, R150, R152, R154, R156, R157, R160, R162, R172, R73, R76, R78, R79, R82, R83, R84, R85, R88: ~, Resistor_SMD:R_0603_1608Metric
- removed R122, R123, R129, R132, R133, R135, R138, R140, R142, R144, R145, R148, R149, R151, R153, R155, R158, R159, R163, R166, R167, R74, R75, R77, R80, R87: 4.7k, Resistor_SMD:R_0603_1608Metric
- removed R124, R126: 470R, Resistor_SMD:R_0603_1608Metric
- removed the R13 at (22.1, -69.8)
- removed the R13 at (131.5, -69.1)
- removed the R14 at (22.1, -68.3)
- removed the R14 at (131.5, -67.6)
- removed the R15 at (130.3, -50.1)
- removed the R15 at (20.8, -50.8)
- removed R164: 910k, Resistor_SMD:R_0603_1608Metric
- removed the R20 at (130.3, -51.6)
- removed the R20 at (20.8, -52.3)
- removed the R3 at (130.3, -54.7)
- removed the R3 at (20.8, -55.4)
- removed the R34 at (131.5, -63.0)
- removed the R34 at (22.1, -63.8)
- removed the R35 at (131.5, -64.6)
- removed the R35 at (22.1, -65.3)
- removed R53, R54, R55, R56, R57, R58, R59, R60, R61: 75R, Resistor_SMD:R_0603_1608Metric
- removed R62, R63, R64, R65, R66, R67: 330R, Resistor_SMD:R_0603_1608Metric
- removed R89: 5.1k, Resistor_SMD:R_0603_1608Metric
- removed R91, R92, R93, R94, R95, R96, R97: 22R, Resistor_SMD:R_0603_1608Metric
- removed RN1: 4D03WGJ0102T5E, Resistor_SMD:R_Array_Convex_4x0603
- removed SW2, SW3, SW4: TS-1187A-B-A-B, Button_Switch_SMD:SW_SPST_TL3342
- removed TP11, TP12, TP13, TP14, TP15, TP16, TP17, TP18, TP19, TP20, TP21, TP22, TP23, TP24, TP25, TP26, TP27, TP28, TP29, TP30, TP31, TP32, TP33, TP34: TestPoint, TestPoint:TestPoint_Pad_D1.0mm
- removed TR3: H2450G, MAS_Package_nostd:Transformer_Ethernet_E-NETTR_24
- removed U10: W25Q256FVEIG, MAS_Package_std:WSON-8-1EP_8x6mm_P1.27mm_EP3.4x4mm
- removed U11: MT7603E, MAS_Package_std:QFN-56-1EP_7x7mm_P0.4mm_EP4.6x4.6mm
- removed U12, U13, U14: TPD2EUSB30, Package_TO_SOT_SMD:Texas_DRT-3
- removed U15: IP5328P, Package_DFN_QFN:QFN-40-1EP_6x6mm_P0.5mm_EP4.6x4.6mm
- removed U16: N096-2864KSWEG01-H30, MAS_Package_nostd:SSD1306-oled-0.96
- removed the U2 at (29.3, -48.5)
- removed the U2 at (138.8, -47.8)
- removed U7, U8: MT3420B, Package_TO_SOT_SMD:SOT-23-6
- removed U9 (x2): NT5CB64M16FP-DH (!), Package_BGA:BGA-96_9.0x13.0mm_Layout2x3x16_P0.8mm
- removed X1: HSO321S-50MHZ-3.3V, MAS_Package_std:Oscillator_SMD_SMD3225-4P
- removed the Y1 at (150.1, -48.2)
- removed the Y1 at (40.6, -48.9)
- added C57: 10n, Capacitor_SMD:C_0603_1608Metric, F.Cu at (156.4, -51.3)
- added C58: 10n, Capacitor_SMD:C_0603_1608Metric, F.Cu at (156.4, -48.8)
- added C59: 10n, Capacitor_SMD:C_0603_1608Metric, F.Cu at (156.4, -46.3)
- added C60: 10n, Capacitor_SMD:C_0603_1608Metric, F.Cu at (156.4, -43.8)
- added C61: 10n, Capacitor_SMD:C_0603_1608Metric, F.Cu at (156.4, -41.2)
- added C62: 10n, Capacitor_SMD:C_0603_1608Metric, F.Cu at (156.4, -38.7)
- added C63: 10n, Capacitor_SMD:C_0603_1608Metric, F.Cu at (156.4, -36.2)
- added C64: 22p, Capacitor_SMD:C_0603_1608Metric, F.Cu at (156.4, -33.7)
- added C65: 22p, Capacitor_SMD:C_0603_1608Metric, F.Cu at (160.4, -61.3)
- added C66: 10n, Capacitor_SMD:C_0603_1608Metric, F.Cu at (160.4, -58.8)
- added C67: 10n, Capacitor_SMD:C_0603_1608Metric, F.Cu at (160.4, -56.3)
- added C68: 100n, Capacitor_SMD:C_0603_1608Metric, F.Cu at (160.4, -53.8)
- added C69: 100n, Capacitor_SMD:C_0603_1608Metric, F.Cu at (160.4, -51.3)
- added C70: 10n, Capacitor_SMD:C_0603_1608Metric, F.Cu at (160.4, -48.8)
- added C71: 10n, Capacitor_SMD:C_0603_1608Metric, F.Cu at (160.4, -46.3)
- added C72: 10u, Capacitor_SMD:C_0805_2012Metric, F.Cu at (161.9, -18.9)
- added C73: 10u, Capacitor_SMD:C_0805_2012Metric, F.Cu at (161.9, -15.9)
- added C74: 10n, Capacitor_SMD:C_0603_1608Metric, F.Cu at (160.4, -43.8)
- added C75: 10n, Capacitor_SMD:C_0603_1608Metric, F.Cu at (160.4, -41.2)
- added C76: 22u, Capacitor_SMD:C_0805_2012Metric, F.Cu at (161.9, -12.9)
- added D4: STPS2L40U, Diode_SMD:D_SMB, F.Cu at (196.0, -17.8)
- added R10: 75R, Resistor_SMD:R_0603_1608Metric, F.Cu at (168.4, -48.8)
- added R11: 75R, Resistor_SMD:R_0603_1608Metric, F.Cu at (168.4, -46.3)
- added R13: 75R, Resistor_SMD:R_0603_1608Metric, F.Cu at (168.4, -41.2)
- added R14: 75R, Resistor_SMD:R_0603_1608Metric, F.Cu at (168.4, -38.7)
- added R15: 75R, Resistor_SMD:R_0603_1608Metric, F.Cu at (168.4, -36.2)
- added R20: 0.5R, Resistor_SMD:R_0603_1608Metric, F.Cu at (172.4, -53.8)
- added R3: 75R, Resistor_SMD:R_0603_1608Metric, F.Cu at (164.4, -36.2)
- added R34: 4.7k, Resistor_SMD:R_0603_1608Metric, F.Cu at (176.4, -56.3)
- added R35: 4.7k, Resistor_SMD:R_0603_1608Metric, F.Cu at (176.4, -53.8)
- added U2: AT24C16, Package_SO:SOIC-8_3.9x4.9mm_P1.27mm, F.Cu at (180.5, -29.2)
- added Y1: SX3B25.000F1510F30, MAS_Package_std:Oscillator_SMD_SMD3225-4P, F.Cu at (203.6, -47.9)
- C1, C23, C4, C5, C6, C7: value 10u -> 100n; footprint Capacitor_SMD:C_0805_2012Metric -> Capacitor_SMD:C_0603_1608Metric
- C14, C15, C30: value 2.2u -> 100n; footprint Capacitor_SMD:C_0805_2012Metric -> Capacitor_SMD:C_0603_1608Metric
- C17: value 10u -> 1n
- C18, C19, C20: value 100n -> 1n; footprint Capacitor_SMD:C_0603_1608Metric -> Capacitor_SMD:C_0805_2012Metric
- C21, C22: value 100n -> 27p
- C24: value 4.7p -> 10u; footprint Capacitor_SMD:C_0603_1608Metric -> Capacitor_Tantalum_SMD:CP_EIA-7343-31_Kemet-D
- C25: value 4.7p -> 10u; footprint Capacitor_SMD:C_0603_1608Metric -> Capacitor_SMD:C_0805_2012Metric
- C26: value 100n -> 10u; footprint Capacitor_SMD:C_0603_1608Metric -> Capacitor_Tantalum_SMD:CP_EIA-7343-31_Kemet-D
- C27, C50: value 100n -> 10u; footprint Capacitor_SMD:C_0603_1608Metric -> Capacitor_SMD:C_0805_2012Metric
- C28: value 100n -> 2.2u; footprint Capacitor_SMD:C_0603_1608Metric -> Capacitor_SMD:C_1206_3216Metric
- C29: value 100n -> 470p; footprint Capacitor_SMD:C_0603_1608Metric -> Capacitor_SMD:C_0805_2012Metric
- C31, C32, C33: value 2.2u -> 22u
- C34: value 100u -> 4.7u; footprint Capacitor_Tantalum_SMD:CP_EIA-7343-31_Kemet-D -> Capacitor_SMD:C_0805_2012Metric
- C35: value 100uF -> 4.7u; footprint Capacitor_Tantalum_SMD:CP_EIA-3528-21_Kemet-B -> Capacitor_SMD:C_0805_2012Metric
- C36: value 10u -> 4.7u
- C37, C48: value 10u -> 22u
- C38, C39, C44, C49, C77, C80, C86, C87: value 100n -> 22u; footprint Capacitor_SMD:C_0603_1608Metric -> Capacitor_SMD:C_0805_2012Metric
- C40: value 22p -> 100n; footprint Capacitor_SMD:C_0603_1608Metric -> Capacitor_SMD:C_0805_2012Metric
- C41: value 22p -> 4.7u; footprint Capacitor_SMD:C_0603_1608Metric -> Capacitor_SMD:C_0805_2012Metric
- C42, C43: value 100n -> 4.7u; footprint Capacitor_SMD:C_0603_1608Metric -> Capacitor_SMD:C_0805_2012Metric
- C45, C46, C47: value 10u -> 1n; footprint Capacitor_SMD:C_0805_2012Metric -> Capacitor_SMD:C_0603_1608Metric
- C51: value 22p -> 10u; footprint Capacitor_SMD:C_0603_1608Metric -> Capacitor_SMD:C_0805_2012Metric
- C52: value 22p -> 100n
- C54, C78, C79, C83, C84, C88, C89: value 100n -> 10n
- C55, C56: value 10u -> 10n; footprint Capacitor_SMD:C_0805_2012Metric -> Capacitor_SMD:C_0603_1608Metric
- C81: value 4.7u -> 22u
- C82, C85: value 4.7u -> 10n; footprint Capacitor_SMD:C_0805_2012Metric -> Capacitor_SMD:C_0603_1608Metric
- D1: value LEDY -> STPS2L40U; footprint Diode_SMD:D_0603_1608Metric -> Diode_SMD:D_SMB
- D2: value LEDG -> MBR0540; footprint Diode_SMD:D_0603_1608Metric -> Diode_SMD:D_SOD-123
- D3: value MBR0540 -> STPS2L40U; footprint Diode_SMD:D_SOD-123 -> Diode_SMD:D_SMB
- F1: moved to F.Cu
- J1: value DS1128-09-S8B8X -> RJ45-B-1*4; footprint MAS_Package_std:RJ45_DS1128-09-S8B8X -> MAS_Package_std:RJ45_B_1_4; moved to F.Cu
- J2: value DS1128-09-S8B8X -> TYPE-C-31-M-12; footprint MAS_Package_std:RJ45_DS1128-09-S8B8X -> MAS_Package_std:USB_C_Receptacle_HRO_TYPE-C-31-M-12; moved to F.Cu
- J3: value DS1128-09-S8B8X -> 98424-G52-06ALF; footprint MAS_Package_std:RJ45_DS1128-09-S8B8X -> Connector_PinSocket_2.00mm:PinSocket_2x03_P2.00mm_Vertical_SMD; moved to F.Cu
- L1: value SLO0530H2R2MTT -> SLO0530H1R0MTT
- L2: value SLO0530H1R0MTT -> SMMS0650; footprint MAS_Package_std:Power_inductor_SMD_0530 -> MAS_Package_nostd:SMDL_7.1x6.6x5mm
- L4, L5: value SLO0530H2R2MTT -> CBM160808U121T; footprint MAS_Package_std:Power_inductor_SMD_0530 -> Inductor_SMD:L_0603_1608Metric
- R1, R12, R16, R6, R7: value 1k -> 75R
- R17: value 100k -> 22k
- R18: value 10k -> 22k
- R19: value 1.1k -> 2.49k
- R2: value 240R -> 75R
- R21: value 330k -> 4.7k
- R22: value 51k -> 4.7k
- R23: value 2k -> 4.7k
- R24: value 68k -> ~
- R25: value 68k -> 0.33R; footprint Resistor_SMD:R_0603_1608Metric -> Resistor_SMD:R_1206_3216Metric
- R27: value 100k -> 0.5R
- R28: value 100k -> 3.6k; footprint Resistor_SMD:R_0603_1608Metric -> Resistor_SMD:R_0805_2012Metric
- R29: value 120k -> 1.2k; footprint Resistor_SMD:R_0603_1608Metric -> Resistor_SMD:R_0805_2012Metric
- R30, R32, R33, R36, R37, R39: value 100k -> 4.7k
- R31, R38: value 150k -> 4.7k
- R4, R9: value 10k -> 75R
- R40, R41, R46: value ~ -> 4.7k
- R44, R45: value 1k -> 4.7k
- R47: value 24k -> 100k
- R48: value 4.7k -> 100k
- R49: value ~ -> 100k
- R5: value 470R -> 75R
- R50: value 75R -> 120k
- R51: value 75R -> 100k
- R52: value 75R -> 22k
- R8: value ~ -> 75R
- SW1: value TS-1187A-B-A-B -> SK-12D02-G040; footprint Button_Switch_SMD:SW_SPST_TL3342 -> MAS_Package_std:SW_Slide_SK-12D02-G040
- TR1, TR2: value H2450G -> 82FB-02NL; footprint MAS_Package_nostd:Transformer_Ethernet_E-NETTR_24 -> MAS_Package_nostd:Transformer_Ethernet_YDS-Tech_82FB-02NL
- U1: value SN74LVC1G175 -> RTL8370Nx; footprint Package_TO_SOT_SMD:SOT-23-6 -> MAS_Package_std:LQFP-128_14x20mm_P0.5mm
- U3: value TPS63020 -> IP5306; footprint Package_DFN_QFN:DFN-14-1EP_3x4mm_P0.5mm_EP1.7x3.3mm -> MAS_Package_std:SOIC-8-1EP_3.9x4.9mm_P1.27mm_EP2.29x3mm
- U4: value TPS63020 -> MC34063AD; footprint Package_DFN_QFN:DFN-14-1EP_3x4mm_P0.5mm_EP1.7x3.3mm -> Package_SO:SOIC-8_3.9x4.9mm_P1.27mm
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Connections:
- C1 pad 1: +1V1 -> GND
- C1 pad 2: -BATT -> Net-(TR1A-TCT1)
- C10 pad 1: +1V1 -> GND
- C10 pad 2: -BATT -> Net-(TR2A-TCT2)
- C11 pad 1: +1V5 -> GND
- C11 pad 2: -BATT -> Net-(TR2A-TCT3)
- C12 pad 1: +1V0 -> GND
- C12 pad 2: -BATT -> Net-(TR2A-TCT4)
- C13 pad 1: +1V1 -> GND
- C13 pad 2: -BATT -> Net-(TR2B-TCT1)
- C14 pad 1: VD -> GND
- C14 pad 2: -BATT -> Net-(TR2B-TCT2)
- C15 pad 1: VD -> GND
- C15 pad 2: -BATT -> Net-(TR2B-TCT3)
- C16 pad 1: +1V5 -> GND
- C16 pad 2: -BATT -> Net-(TR2B-TCT4)
- C17 pad 1: +1V0 -> GNDREF
- C17 pad 2: -BATT -> Net-(C17-Pad2)
- C18 pad 1: VD -> GNDREF
- C18 pad 2: -BATT -> Net-(C18-Pad2)
- C19 pad 1: VD -> GNDREF
- C19 pad 2: -BATT -> Net-(C19-Pad2)
- C2 pad 1: +BATT -> GND
- C2 pad 2: -BATT -> Net-(TR1A-TCT2)
- C20 pad 1: Net-(C20-Pad1) -> GNDREF
- C20 pad 2: -BATT -> Net-(C20-Pad2)
- C21 pad 1: Net-(C21-Pad1) -> GND
- C21 pad 2: -BATT -> Net-(U1K-XTALI)
- C22 pad 1: +1V1 -> Net-(U1K-XTALO)
- C22 pad 2: -BATT -> GND
- C23 pad 1: +1V5 -> GND
- C23 pad 2: -BATT -> +3V3
- C24 pad 1: Net-(C24-Pad1) -> +24V
- C24 pad 2: Net-(C24-Pad2) -> GND
- C25 pad 2: Net-(C25-Pad2) -> GND
- C26 pad 1: +1V1 -> +24V
- C26 pad 2: -BATT -> GND
- C27 pad 1: +1V1 -> Net-(U3-VIN)
- C27 pad 2: -BATT -> GND
- C28 pad 1: Net-(C28-Pad1) -> +24V
- C28 pad 2: -BATT -> GND
- C29 pad 1: Net-(C29-Pad1) -> Net-(U4-TC)
- C29 pad 2: -BATT -> GND
- C3 pad 1: +1V5 -> GND
- C3 pad 2: -BATT -> Net-(TR1A-TCT3)
- C30 pad 1: Net-(C28-Pad1) -> Net-(D2-A)
- C30 pad 2: -BATT -> GND
- C31 pad 1: Net-(C29-Pad1) -> Net-(U3-BAT)
- C31 pad 2: -BATT -> GND
- C32 pad 1: Net-(C28-Pad1) -> Net-(D4-A)
- C32 pad 2: -BATT -> GND
- C33 pad 1: Net-(C29-Pad1) -> +5C
- C33 pad 2: -BATT -> GND
- C34 pad 1: Net-(C28-Pad1) -> +1V1
- C34 pad 2: -BATT -> GND
- C35 pad 1: Net-(C29-Pad1) -> +1V1
- C35 pad 2: -BATT -> GND
- C36 pad 1: +3V3 -> +1V1
- C36 pad 2: -BATT -> GND
- C37 pad 1: +3V3 -> Net-(D4-K)
- C37 pad 2: -BATT -> GND
- C38 pad 1: +3V3 -> +5C
- C38 pad 2: -BATT -> GND
- C39 pad 1: +3V3 -> Net-(D4-K)
- C39 pad 2: -BATT -> GND
- C4 pad 1: VD -> GND
- C4 pad 2: -BATT -> Net-(TR1A-TCT4)
- C40 pad 1: Net-(C40-Pad1) -> +5C
- C40 pad 2: Net-(C40-Pad2) -> GND
- C41 pad 2: Net-(C41-Pad2) -> GND
- C42 pad 1: +1V1 -> Net-(U1J-PLLVDDL0)
- C42 pad 2: -BATT -> GND
- C43 pad 1: Net-(C40-Pad1) -> Net-(U1J-PLLVDDL1)
- C43 pad 2: -BATT -> GND
- C44 pad 1: Net-(C41-Pad1) -> Net-(D4-K)
- C44 pad 2: -BATT -> GND
- C45 pad 1: Net-(C40-Pad1) -> Net-(C41-Pad1)
- C45 pad 2: -BATT -> GND
- C46 pad 1: Net-(C41-Pad1) -> Net-(U1J-PLLVDDL0)
- C46 pad 2: -BATT -> GND
- C47 pad 1: +3V3 -> Net-(U1J-PLLVDDL1)
- C47 pad 2: -BATT -> GND
- C48 pad 1: +3V3 -> +5V
- C48 pad 2: -BATT -> GND
- C49 pad 1: +3V3 -> +5V
- C49 pad 2: -BATT -> GND
- C5 pad 1: VD -> GND
- C5 pad 2: -BATT -> Net-(TR1B-TCT1)
- C50 pad 1: +3V3 -> +5V
- C50 pad 2: -BATT -> GND
- C51 pad 1: Net-(C51-Pad1) -> +5V
- C51 pad 2: Net-(C51-Pad2) -> GND
- C52 pad 1: Net-(C52-Pad1) -> +5V
- C52 pad 2: Net-(C52-Pad2) -> GND
- C53 pad 1: Net-(C51-Pad1) -> +5V
- C53 pad 2: -BATT -> GND
- C54 pad 1: Net-(C52-Pad1) -> +3V3
- C54 pad 2: -BATT -> GND
- C55 pad 1: Net-(C51-Pad1) -> +1V1
- C55 pad 2: -BATT -> GND
- C56 pad 1: Net-(C52-Pad1) -> +3V3
- C56 pad 2: -BATT -> GND
- C6 pad 1: VD -> GND
- C6 pad 2: -BATT -> Net-(TR1B-TCT2)
- C7 pad 1: VD -> GND
- C7 pad 2: -BATT -> Net-(TR1B-TCT3)
- C77 pad 1: +3V3 -> Net-(JP2-B)
- C77 pad 2: -BATT -> GND
- C78 pad 1: Net-(C78-Pad1) -> +3V3
- C78 pad 2: -BATT -> GND
- C79 pad 1: Net-(C79-Pad1) -> +1V1
- C79 pad 2: -BATT -> GND
- C8 pad 1: +1V0 -> GND
- C8 pad 2: -BATT -> Net-(TR1B-TCT4)
- C80 pad 1: Net-(C79-Pad1) -> Net-(JP1-B)
- C80 pad 2: -BATT -> GND
- C81 pad 1: +3V3 -> Net-(JP2-B)
- C81 pad 2: -BATT -> GND
- C82 pad 1: +1V0 -> +3V3
- C82 pad 2: Net-(C102-Pad2) -> GND
- C83 pad 1: Net-(C83-Pad1) -> +1V1
- C83 pad 2: -BATT -> GND
- C84 pad 1: Net-(C83-Pad1) -> +3V3
- C84 pad 2: -BATT -> GND
- C85 pad 1: +1V0 -> +1V1
- C85 pad 2: Net-(C102-Pad2) -> GND
- C86 pad 1: Net-(C83-Pad1) -> Net-(JP1-B)
- C86 pad 2: -BATT -> GND
- C87 pad 1: +1V0 -> Net-(JP2-B)
- C87 pad 2: Net-(C102-Pad2) -> GND
- C88 pad 1: Net-(C83-Pad1) -> +3V3
- C88 pad 2: -BATT -> GND
- C89 pad 1: -BATT -> +1V1
- C89 pad 2: Net-(C89-Pad2) -> GND
- C9 pad 1: Net-(C9-Pad1) -> GND
- C9 pad 2: -BATT -> Net-(TR2A-TCT1)
- D1 pad 1: Net-(D1-Pad1) -> +24V
- D1 pad 2: Net-(D1-Pad2) -> Net-(D1-A)
- D2 pad 1: Net-(D2-Pad1) -> +3V3
- D2 pad 2: Net-(D2-Pad2) -> Net-(D2-A)
- D3 pad 1: +3V3 -> Net-(D3-K)
- D3 pad 2: /Other/D2DB_PORST_N -> GND
- F1 pad 1: Net-(BT1-Pad1) -> Net-(D4-A)
- F1 pad 2: +BATT -> Net-(BT1-+)
- J1 pad 1: Net-(J1-Pad1) -> Net-(J1A-BI_DA+)
- J1 pad 10: Net-(J1-Pad10) -> /G1+
- J1 pad 11: /Ethernet/Y0- -> /Y1-
- J1 pad 12: Net-(J1-Pad12) -> /Y1+
- J1 pad 14: GNDREF -> Net-(J1B-BI_DA+)
- J1 pad 2: Net-(J1-Pad2) -> Net-(J1A-BI_DA-)
- J1 pad 3: Net-(J1-Pad3) -> Net-(J1A-BI_DB+)
- J1 pad 4: Net-(J1-Pad4) -> Net-(J1A-BI_DC+)
- J1 pad 5: Net-(J1-Pad5) -> Net-(J1A-BI_DC-)
- J1 pad 6: Net-(J1-Pad6) -> Net-(J1A-BI_DB-)
- J1 pad 7: Net-(J1-Pad7) -> Net-(J1A-BI_DD+)
- J1 pad 8: Net-(J1-Pad8) -> Net-(J1A-BI_DD-)
- J1 pad 9: /Ethernet/G0- -> /G1-
- J3 pad 1: Net-(J3-Pad1) -> Net-(D1-A)
- J3 pad 2: Net-(J3-Pad2) -> Net-(D1-A)
- J3 pad 3: Net-(J3-Pad3) -> Net-(D1-A)
- J3 pad 4: Net-(J3-Pad4) -> GND
- J3 pad 5: Net-(J3-Pad5) -> GND
- J3 pad 6: Net-(J3-Pad6) -> GND
- JP1 pad 1: /Charger/VMID -> +1V1
- JP1 pad 2: /Charger/VBUS -> Net-(JP1-B)
- JP2 pad 1: +5V -> +3V3
- JP2 pad 2: Net-(C28-Pad1) -> Net-(JP2-B)
- L1 pad 1: Net-(L1-Pad1) -> Net-(U3-SW)
- L1 pad 2: Net-(L1-Pad2) -> Net-(D4-A)
- L2 pad 1: Net-(L2-Pad1) -> Net-(D3-K)
- L2 pad 2: Net-(L2-Pad2) -> +5C
- L3 pad 1: +3V3 -> +1V1
- L3 pad 2: Net-(C83-Pad1) -> Net-(C41-Pad1)
- L4 pad 1: Net-(L4-Pad1) -> +1V1
- L4 pad 2: Net-(C40-Pad1) -> Net-(U1J-PLLVDDL0)
- L5 pad 1: Net-(L5-Pad1) -> +1V1
- L5 pad 2: Net-(C41-Pad1) -> Net-(U1J-PLLVDDL1)
- L6 pad 1: Net-(L6-Pad1) -> Net-(U5-LX)
- L6 pad 2: Net-(C51-Pad1) -> Net-(JP1-B)
- L7 pad 1: Net-(L7-Pad1) -> Net-(U6-LX)
- L7 pad 2: Net-(C52-Pad1) -> Net-(JP2-B)
- R1 pad 1: Net-(R1-Pad1) -> Net-(C17-Pad2)
- R1 pad 2: Net-(C20-Pad1) -> Net-(TR1A-CMT1)
- R12 pad 1: Net-(C9-Pad1) -> Net-(C19-Pad2)
- R12 pad 2: +BATT -> Net-(TR2A-CMT4)
- R16 pad 1: Net-(R16-Pad1) -> Net-(C20-Pad2)
- R16 pad 2: Net-(C21-Pad1) -> Net-(TR2B-CMT4)
- R17 pad 1: Net-(C28-Pad1) -> GND
- R17 pad 2: Net-(R17-Pad2) -> Net-(J2-CC2)
- R18 pad 1: Net-(C24-Pad2) -> GND
- R18 pad 2: Net-(C28-Pad1) -> Net-(J2-CC1)
- R19 pad 1: Net-(C24-Pad2) -> GND
- R19 pad 2: -BATT -> Net-(U1K-MDIREF)
- R2 pad 1: -BATT -> Net-(C17-Pad2)
- R2 pad 2: Net-(R2-Pad2) -> Net-(TR1A-CMT2)
- R21 pad 1: Net-(C25-Pad2) -> Net-(U2-~{WC})
- R21 pad 2: Net-(C29-Pad1) -> +3V3
- R22 pad 1: Net-(C25-Pad2) -> /SCK
- R22 pad 2: Net-(R22-Pad2) -> +3V3
- R23 pad 1: Net-(R22-Pad2) -> /SDA
- R23 pad 2: -BATT -> +3V3
- R24 pad 1: Net-(C28-Pad1) -> GND
- R24 pad 2: Net-(C24-Pad1) -> Net-(U1K-ATESTCK0)
- R25 pad 1: Net-(C29-Pad1) -> Net-(U4-DC)
- R25 pad 2: Net-(C25-Pad1) -> +24V
- R26 pad 1: Net-(R26-Pad1) -> +3V3
- R26 pad 2: +3V3 -> Net-(D2-A)
- R27 pad 1: Net-(R27-Pad1) -> Net-(U3-BAT)
- R27 pad 2: +3V3 -> Net-(D4-A)
- R28 pad 1: Net-(C40-Pad2) -> Net-(U4-Vfb)
- R28 pad 2: Net-(C40-Pad1) -> +5C
- R29 pad 1: -BATT -> GND
- R29 pad 2: Net-(C40-Pad2) -> Net-(U4-Vfb)
- R30 pad 1: Net-(C41-Pad2) -> Net-(U1I-P6LED0/GPIO1)
- R30 pad 2: Net-(C41-Pad1) -> +3V3
- R31 pad 1: -BATT -> Net-(U1I-P6LED1/GPIO7)
- R31 pad 2: Net-(C41-Pad2) -> +3V3
- R32 pad 1: Net-(R32-Pad1) -> Net-(U1I-P5LED0)
- R33 pad 1: Net-(R33-Pad1) -> Net-(U1I-P5LED1)
- R36 pad 1: Net-(C51-Pad2) -> Net-(U1I-P3LED2/SLED_P3B/STRP_EN_PWRLIGHT)
- R36 pad 2: Net-(C51-Pad1) -> +3V3
- R37 pad 1: -BATT -> Net-(U1I-P3LED0/SLED_P2B/STRP_EN_FLASH)
- R37 pad 2: Net-(C51-Pad2) -> GND
- R38 pad 1: Net-(C52-Pad2) -> Net-(U1I-P2LED2/SLED_P1B/STRP_DIS_8051)
- R38 pad 2: Net-(C52-Pad1) -> +3V3
- R39 pad 1: -BATT -> Net-(U1I-P2LED0/SLED_P0B/STRP_DISAUTOLOAD)
- R39 pad 2: Net-(C52-Pad2) -> GND
- R4 pad 1: +BATT -> Net-(C17-Pad2)
- R4 pad 2: Net-(Q2-Pad3) -> Net-(TR1A-CMT4)
- R40 pad 1: -BATT -> Net-(U1I-P2LED1/SLED_G1B/GPIO4)
- R40 pad 2: /Memory/ND_D4 -> +3V3
- R41 pad 1: /Memory/ND_CS_N -> Net-(U1I-P1LED2/SLED_P3_7A/STRP_SMI_SEL_1)
- R42 pad 1: /Memory/ND_D7 -> Net-(U1I-P1LED0/SLED_P2_6A/STRP_MID29)
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Routing:
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- removed copper zone on B.Cu, net -BATT
- removed copper zone on F.Cu, net -BATT
Other:
- board size 88 x 111 mm -> 84 x 50 mm
- copper layers 4 -> 2

Commit message: Update main.kicad_pcb
Parts:
- moved TP3 200.5 mm to (1.39, -15.0), turned to -90 degrees
- moved R17 198.0 mm to (-10.7, 13.9), turned to 180 degrees
- moved R18 196.1 mm to (-10.7, 11.4), turned to 180 degrees
- moved D4 183.8 mm to (12.2, -12.7), turned to -90 degrees
- moved R48 183.6 mm to (13.2, 24.4)
- moved R52 177.4 mm to (13.2, 18.0)
- moved U3 177.2 mm to (3.30, -20.4), turned to -90 degrees
- moved R51 177.0 mm to (13.2, 14.2), turned to 180 degrees
- moved R47 171.9 mm to (27.3, 24.4)
- moved R27 171.2 mm to (2.91, -15.0), turned to -90 degrees
- moved L7 168.0 mm to (8.13, 19.3), turned to 90 degrees
- moved C87 167.6 mm to (3.68, 21.2), turned to -90 degrees
- moved C77 167.5 mm to (4.95, 13.6), turned to 90 degrees
- moved L1 166.6 mm to (6.60, -12.9), turned to -90 degrees
- moved R20 166.6 mm to (8.12, -26.4)
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
Commit message: The layout of the board
Parts:
- added BT1: BH-18650-B1BA002, MAS_Package_nostd:BatteryHolder_BH-18650-B1BA002, F.Cu at (37.6, 58.9)
- added C90: 10n, Capacitor_SMD:C_0402_1005Metric, B.Cu at (33.3, -16.2)
- C1, C10, C11, C12, C13, C14, C15, C16, C2, C21, C22, C3, C4, C5, C54, C55, C56, C57, C58, C59, C6, C60, C61, C62, C63, C66, C67, C7, C70, C71, C74, C75, C78, C79, C8, C83, C84, C85, C88, C89, C9: footprint Capacitor_SMD:C_0603_1608Metric -> Capacitor_SMD:C_0402_1005Metric; moved to B.Cu
- C17, C18, C19, C20, C28, C33, C34, C38, C40, C41, D1, D3, L2, L3, R25, R28, R29, U4, Y1: moved to B.Cu
- C23, C30, C45, C46, C47, C52, C53, C68, C69, C82: footprint Capacitor_SMD:C_0603_1608Metric -> Capacitor_SMD:C_0402_1005Metric
- C24, C26: value 10u -> 2.2u; footprint Capacitor_Tantalum_SMD:CP_EIA-7343-31_Kemet-D -> Capacitor_SMD:C_1206_3216Metric; moved to B.Cu
- C29: value 470p -> 150p; moved to B.Cu
- D4: value STPS2L40U -> MBR0540; footprint Diode_SMD:D_SMB -> Diode_SMD:D_SOD-123
- JP1, JP2: value J_Boot -> jump
- R1, R10, R11, R12, R13, R14, R15, R16, R2, R3, R30, R31, R32, R33, R34, R35, R36, R37, R38, R39, R4, R40, R41, R42, R43, R44, R45, R46, R5, R6, R7, R8, R9: footprint Resistor_SMD:R_0603_1608Metric -> Resistor_SMD:R_0402_1005Metric; moved to B.Cu
- R17, R18, R19, R21, R22, R23, R24, R26, R47, R48, R49, R51, R52: footprint Resistor_SMD:R_0603_1608Metric -> Resistor_SMD:R_0402_1005Metric
- TP1, TP10, TP2, TP3, TP4, TP5, TP6, TP7, TP8, TP9: footprint TestPoint:TestPoint_Pad_D1.0mm -> MAS_Package_std:TestPoint_Pad_D0.5mm
- TR1, TR2: value 82FB-02NL -> G5002CG; footprint MAS_Package_nostd:Transformer_Ethernet_YDS-Tech_82FB-02NL -> MAS_Package_nostd:Transformer_Ethernet_YDS-Tech_G5002CG
- moved R30 171.8 mm to (31.8, -1.52), turned to -90 degrees
- moved R31 170.0 mm to (32.8, -1.52), turned to -90 degrees
- moved R32 167.7 mm to (33.8, -1.52), turned to -90 degrees
- moved R33 166.0 mm to (34.8, -1.53), turned to -90 degrees
- moved R34 164.2 mm to (35.8, -1.52), turned to -90 degrees
- moved R35 162.5 mm to (36.8, -1.52), turned to -90 degrees
- moved R36 160.8 mm to (37.8, -1.52), turned to -90 degrees
- moved R37 159.1 mm to (38.9, -1.52), turned to -90 degrees
- moved R38 157.5 mm to (39.9, -1.52), turned to -90 degrees
- moved R39 155.8 mm to (40.9, -1.52), turned to -90 degrees
- moved R40 154.3 mm to (41.9, -1.52), turned to -90 degrees
- moved R41 152.7 mm to (42.9, -1.53), turned to -90 degrees
- moved R42 151.2 mm to (43.9, -1.53), turned to -90 degrees
- moved R43 149.7 mm to (45.0, -1.52), turned to -90 degrees
- moved R44 148.4 mm to (46.0, -1.53), turned to -90 degrees
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Connections:
- C1 pad 2: Net-(TR1A-TCT1) -> Net-(TR1A-TCT4)
- C10 pad 2: Net-(TR2A-TCT2) -> Net-(TR2A-TCT3)
- C11 pad 2: Net-(TR2A-TCT3) -> Net-(TR2A-TCT2)
- C12 pad 2: Net-(TR2A-TCT4) -> Net-(TR2A-TCT1)
- C13 pad 2: Net-(TR2B-TCT1) -> Net-(TR2B-TCT4)
- C14 pad 2: Net-(TR2B-TCT2) -> Net-(TR2B-TCT3)
- C15 pad 2: Net-(TR2B-TCT3) -> Net-(TR2B-TCT2)
- C16 pad 2: Net-(TR2B-TCT4) -> Net-(TR2B-TCT1)
- C2 pad 2: Net-(TR1A-TCT2) -> Net-(TR1A-TCT3)
- C3 pad 2: Net-(TR1A-TCT3) -> Net-(TR1A-TCT2)
- C4 pad 2: Net-(TR1A-TCT4) -> Net-(TR1A-TCT1)
- C5 pad 2: Net-(TR1B-TCT1) -> Net-(TR1B-TCT4)
- C6 pad 2: Net-(TR1B-TCT2) -> Net-(TR1B-TCT3)
- C7 pad 2: Net-(TR1B-TCT3) -> Net-(TR1B-TCT2)
- C8 pad 2: Net-(TR1B-TCT4) -> Net-(TR1B-TCT1)
- C9 pad 2: Net-(TR2A-TCT1) -> Net-(TR2A-TCT4)
- R1 pad 2: Net-(TR1A-CMT1) -> Net-(TR1A-CMT4)
- R10 pad 2: Net-(TR2A-CMT2) -> Net-(TR2A-CMT3)
- R11 pad 2: Net-(TR2A-CMT3) -> Net-(TR2A-CMT2)
- R12 pad 2: Net-(TR2A-CMT4) -> Net-(TR2A-CMT1)
- R13 pad 2: Net-(TR2B-CMT1) -> Net-(TR2B-CMT4)
- R14 pad 2: Net-(TR2B-CMT2) -> Net-(TR2B-CMT3)
- R15 pad 2: Net-(TR2B-CMT3) -> Net-(TR2B-CMT2)
- R16 pad 2: Net-(TR2B-CMT4) -> Net-(TR2B-CMT1)
- R2 pad 2: Net-(TR1A-CMT2) -> Net-(TR1A-CMT3)
- R3 pad 2: Net-(TR1A-CMT3) -> Net-(TR1A-CMT2)
- R4 pad 2: Net-(TR1A-CMT4) -> Net-(TR1A-CMT1)
- R5 pad 2: Net-(TR1B-CMT1) -> Net-(TR1B-CMT4)
- R6 pad 2: Net-(TR1B-CMT2) -> Net-(TR1B-CMT3)
- R7 pad 2: Net-(TR1B-CMT3) -> Net-(TR1B-CMT2)
- R8 pad 2: Net-(TR1B-CMT4) -> Net-(TR1B-CMT1)
- R9 pad 2: Net-(TR2A-CMT1) -> Net-(TR2A-CMT4)
- TR1 pad 1: Net-(TR1A-TCT1) -> Net-(TR1A-TD1+)
- TR1 pad 10: Net-(TR1A-TCT4) -> Net-(TR1A-TD4+)
- TR1 pad 11: Net-(TR1A-TD4+) -> Net-(TR1A-TCT4)
- TR1 pad 13: Net-(TR1B-TCT1) -> (no net)
- TR1 pad 15: Net-(TR1B-TD1-) -> Net-(TR1B-TCT1)
- TR1 pad 16: Net-(TR1B-TCT2) -> Net-(TR1B-TD1-)
- TR1 pad 18: Net-(TR1B-TD2-) -> Net-(TR1B-TCT2)
- TR1 pad 19: Net-(TR1B-TCT3) -> Net-(TR1B-TD2-)
- TR1 pad 2: Net-(TR1A-TD1+) -> Net-(TR1A-TCT1)
- TR1 pad 21: Net-(TR1B-TD3-) -> Net-(TR1B-TCT3)
- TR1 pad 22: Net-(TR1B-TCT4) -> Net-(TR1B-TD3-)
- TR1 pad 24: Net-(TR1B-TD4-) -> Net-(TR1B-TCT4)
- TR1 pad 25: Net-(J1B-BI_DA+) -> Net-(TR1B-TD4-)
- TR1 pad 26: Net-(J1B-BI_DA-) -> Net-(J1B-BI_DD-)
- TR1 pad 28: Net-(J1B-BI_DC+) -> Net-(J1B-BI_DD+)
- TR1 pad 29: Net-(J1B-BI_DC-) -> Net-(J1B-BI_DB+)
- TR1 pad 31: Net-(J1B-BI_DB+) -> Net-(J1B-BI_DB-)
- TR1 pad 32: Net-(J1B-BI_DB-) -> Net-(J1B-BI_DC-)
- TR1 pad 34: Net-(J1B-BI_DD+) -> Net-(J1B-BI_DC+)
- TR1 pad 35: Net-(J1B-BI_DD-) -> Net-(J1B-BI_DA+)
- TR1 pad 37: Net-(J1A-BI_DA+) -> Net-(J1B-BI_DA-)
- TR1 pad 38: Net-(J1A-BI_DA-) -> (no net)
- TR1 pad 39: Net-(TR1A-CMT4) -> Net-(J1A-BI_DD-)
- TR1 pad 4: Net-(TR1A-TCT2) -> Net-(TR1A-TD2+)
- TR1 pad 40: Net-(J1A-BI_DC+) -> Net-(TR1A-CMT4)
- TR1 pad 41: Net-(J1A-BI_DC-) -> Net-(J1A-BI_DD+)
- TR1 pad 42: Net-(TR1A-CMT3) -> Net-(J1A-BI_DB+)
- TR1 pad 43: Net-(J1A-BI_DB+) -> Net-(TR1A-CMT3)
- TR1 pad 45: Net-(TR1A-CMT2) -> Net-(J1A-BI_DC-)
- TR1 pad 46: Net-(J1A-BI_DD+) -> Net-(TR1A-CMT2)
- TR1 pad 47: Net-(J1A-BI_DD-) -> Net-(J1A-BI_DC+)
- TR1 pad 48: Net-(TR1A-CMT1) -> Net-(J1A-BI_DA+)
- TR1 pad 5: Net-(TR1A-TD2+) -> Net-(TR1A-TCT2)
- TR1 pad 7: Net-(TR1A-TCT3) -> Net-(TR1A-TD3+)
- TR1 pad 8: Net-(TR1A-TD3+) -> Net-(TR1A-TCT3)
- TR2 pad 1: Net-(TR2A-TCT1) -> Net-(TR2A-TD1+)
- TR2 pad 10: Net-(TR2A-TCT4) -> Net-(TR2A-TD4+)
- TR2 pad 11: Net-(TR2A-TD4+) -> Net-(TR2A-TCT4)
- TR2 pad 13: Net-(TR2B-TCT1) -> (no net)
- TR2 pad 15: Net-(TR2B-TD1-) -> Net-(TR2B-TCT1)
- TR2 pad 16: Net-(TR2B-TCT2) -> Net-(TR2B-TD1-)
- TR2 pad 18: Net-(TR2B-TD2-) -> Net-(TR2B-TCT2)
- TR2 pad 19: Net-(TR2B-TCT3) -> Net-(TR2B-TD2-)
- TR2 pad 2: Net-(TR2A-TD1+) -> Net-(TR2A-TCT1)
- TR2 pad 21: Net-(TR2B-TD3-) -> Net-(TR2B-TCT3)
- TR2 pad 22: Net-(TR2B-TCT4) -> Net-(TR2B-TD3-)
- TR2 pad 24: Net-(TR2B-TD4-) -> Net-(TR2B-TCT4)
- TR2 pad 25: Net-(J1D-BI_DA+) -> Net-(TR2B-TD4-)
- TR2 pad 26: Net-(J1D-BI_DA-) -> Net-(J1D-BI_DD-)
- TR2 pad 28: Net-(J1D-BI_DC+) -> Net-(J1D-BI_DD+)
- TR2 pad 29: Net-(J1D-BI_DC-) -> Net-(J1D-BI_DB+)
- TR2 pad 31: Net-(J1D-BI_DB+) -> Net-(J1D-BI_DB-)
- TR2 pad 32: Net-(J1D-BI_DB-) -> Net-(J1D-BI_DC-)
- TR2 pad 34: Net-(J1D-BI_DD+) -> Net-(J1D-BI_DC+)
- TR2 pad 35: Net-(J1D-BI_DD-) -> Net-(J1D-BI_DA+)
- TR2 pad 37: Net-(J1C-BI_DA+) -> Net-(J1D-BI_DA-)
- TR2 pad 38: Net-(J1C-BI_DA-) -> (no net)
- TR2 pad 39: Net-(TR2A-CMT4) -> Net-(J1C-BI_DD-)
- TR2 pad 4: Net-(TR2A-TCT2) -> Net-(TR2A-TD2+)
- TR2 pad 40: Net-(J1C-BI_DC+) -> Net-(TR2A-CMT4)
- TR2 pad 41: Net-(J1C-BI_DC-) -> Net-(J1C-BI_DD+)
- TR2 pad 42: Net-(TR2A-CMT3) -> Net-(J1C-BI_DB+)
- TR2 pad 43: Net-(J1C-BI_DB+) -> Net-(TR2A-CMT3)
- TR2 pad 45: Net-(TR2A-CMT2) -> Net-(J1C-BI_DC-)
- TR2 pad 46: Net-(J1C-BI_DD+) -> Net-(TR2A-CMT2)
- TR2 pad 47: Net-(J1C-BI_DD-) -> Net-(J1C-BI_DC+)
- TR2 pad 48: Net-(TR2A-CMT1) -> Net-(J1C-BI_DA+)
- TR2 pad 5: Net-(TR2A-TD2+) -> Net-(TR2A-TCT2)
- TR2 pad 7: Net-(TR2A-TCT3) -> Net-(TR2A-TD3+)
- TR2 pad 8: Net-(TR2A-TD3+) -> Net-(TR2A-TCT3)
- U1 pad 1: Net-(TR2A-TD3+) -> Net-(TR2B-TD2-)
- U1 pad 103: Net-(TR1A-TD1+) -> (no net)
- U1 pad 104: Net-(TR1A-TD1-) -> (no net)
- U1 pad 105: Net-(TR1A-TD2+) -> (no net)
- U1 pad 106: Net-(TR1A-TD2-) -> (no net)
- U1 pad 108: Net-(TR1A-TD3+) -> (no net)
- U1 pad 109: Net-(TR1A-TD3-) -> (no net)
- U1 pad 11: Net-(TR2B-TD3+) -> Net-(TR2A-TD2-)
- U1 pad 110: Net-(TR1A-TD4+) -> (no net)
- U1 pad 111: Net-(TR1A-TD4-) -> (no net)
- U1 pad 113: Net-(TR1B-TD1+) -> (no net)
- U1 pad 114: Net-(TR1B-TD1-) -> (no net)
- U1 pad 115: Net-(TR1B-TD2+) -> (no net)
- U1 pad 116: Net-(TR1B-TD2-) -> (no net)
- U1 pad 118: Net-(TR1B-TD3+) -> (no net)
- U1 pad 119: Net-(TR1B-TD3-) -> (no net)
- U1 pad 12: Net-(TR2B-TD3-) -> Net-(TR2A-TD2+)
- U1 pad 120: Net-(TR1B-TD4+) -> (no net)
- U1 pad 121: Net-(TR1B-TD4-) -> (no net)
- U1 pad 124: Net-(TR2A-TD1+) -> Net-(TR2B-TD4-)
- U1 pad 125: Net-(TR2A-TD1-) -> Net-(TR2B-TD4+)
- U1 pad 126: Net-(TR2A-TD2+) -> Net-(TR2B-TD3-)
- U1 pad 127: Net-(TR2A-TD2-) -> Net-(TR2B-TD3+)
- U1 pad 13: Net-(TR2B-TD4+) -> Net-(TR2A-TD1-)
- U1 pad 14: Net-(TR2B-TD4-) -> Net-(TR2A-TD1+)
- U1 pad 2: Net-(TR2A-TD3-) -> Net-(TR2B-TD2+)
- U1 pad 25: unconnected-(U1E-P4MDIAP-Pad25) -> Net-(TR1B-TD4-)
- U1 pad 26: unconnected-(U1E-P4MDIAN-Pad26) -> Net-(TR1B-TD4+)
- U1 pad 27: unconnected-(U1E-P4MDIBP-Pad27) -> Net-(TR1B-TD3-)
- U1 pad 28: unconnected-(U1E-P4MDIBN-Pad28) -> Net-(TR1B-TD3+)
- U1 pad 3: Net-(TR2A-TD4+) -> Net-(TR2B-TD1-)
- U1 pad 30: unconnected-(U1E-P4MDICP-Pad30) -> Net-(TR1B-TD2-)
- U1 pad 31: unconnected-(U1E-P4MDICN-Pad31) -> Net-(TR1B-TD2+)
- U1 pad 32: unconnected-(U1E-P4MDIDP-Pad32) -> Net-(TR1B-TD1-)
- U1 pad 33: unconnected-(U1E-P4MDIDN-Pad33) -> Net-(TR1B-TD1+)
- U1 pad 35: unconnected-(U1F-P5MDIAP-Pad35) -> Net-(TR1A-TD4-)
- U1 pad 36: unconnected-(U1F-P5MDIAN-Pad36) -> Net-(TR1A-TD4+)
- U1 pad 37: unconnected-(U1F-P5MDIBP-Pad37) -> Net-(TR1A-TD3-)
- U1 pad 38: unconnected-(U1F-P5MDIBN-Pad38) -> Net-(TR1A-TD3+)
- U1 pad 4: Net-(TR2A-TD4-) -> Net-(TR2B-TD1+)
- U1 pad 40: unconnected-(U1F-P5MDICP-Pad40) -> Net-(TR1A-TD2-)
- U1 pad 41: unconnected-(U1F-P5MDICN-Pad41) -> Net-(TR1A-TD2+)
- U1 pad 42: unconnected-(U1F-P5MDIDP-Pad42) -> Net-(TR1A-TD1-)
- U1 pad 43: unconnected-(U1F-P5MDIDN-Pad43) -> Net-(TR1A-TD1+)
- U1 pad 6: Net-(TR2B-TD1+) -> Net-(TR2A-TD4-)
- U1 pad 7: Net-(TR2B-TD1-) -> Net-(TR2A-TD4+)
- U1 pad 8: Net-(TR2B-TD2+) -> Net-(TR2A-TD3-)
- U1 pad 9: Net-(TR2B-TD2-) -> Net-(TR2A-TD3+)

Commit message: update sch and pcb
Parts:
- removed BT1: BH-18650-B1BA002, MAS_Package_nostd:BatteryHolder_BH-18650-B1BA002
- added J4: batt, Connector_PinHeader_2.54mm:PinHeader_1x02_P2.54mm_Vertical, F.Cu at (13.5, -17.8)
- C24, C26, C28, C33, C38, C40, L2, U4: moved to F.Cu
- C29: footprint Capacitor_SMD:C_0805_2012Metric -> Capacitor_SMD:C_0603_1608Metric; moved to F.Cu
- D1, D3: value STPS2L40U -> SS14; footprint Diode_SMD:D_SMB -> Diode_SMD:D_SMA; moved to F.Cu
- R17, R18: moved to B.Cu
- R25: value 0.33R -> 0.5R; footprint Resistor_SMD:R_1206_3216Metric -> Resistor_SMD:R_0805_2012Metric; moved to F.Cu
- R28, R29: footprint Resistor_SMD:R_0805_2012Metric -> Resistor_SMD:R_0603_1608Metric; moved to F.Cu
- moved C40 77.8 mm to (81.3, -20.1), turned to 0 degrees
- moved C33 74.7 mm to (81.3, -18.0), turned to 0 degrees
- moved C29 73.3 mm to (75.4, -6.28), turned to -90 degrees
- moved R28 70.5 mm to (77.5, -17.8), turned to 0 degrees
- moved C72 70.1 mm to (8.64, -5.08), turned to -90 degrees
- moved L6 69.5 mm to (13.1, -6.60)
- moved C64 69.5 mm to (10.7, -11.7)
- moved R50 69.5 mm to (12.2, -11.7)
- moved U5 69.5 mm to (14.7, -11.7)
- moved R49 69.3 mm to (9.14, -11.4)
- moved R47 69.0 mm to (17.1, -12.8)
- moved C86 68.7 mm to (15.7, -2.03), turned to -90 degrees
- moved C68 68.5 mm to (8.13, -11.4)
- moved C76 68.2 mm to (8.64, -8.64), turned to 90 degrees
- moved R29 67.8 mm to (74.9, -17.8)
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
Commit message: update pcb rules
Other:
- copper layers 2 -> 4
Changed lines of the file:
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@@
   (layers
     (0 "F.Cu" signal)
+    (1 "In1.Cu" signal)
+    (2 "In2.Cu" signal)
     (31 "B.Cu" signal)
     (32 "B.Adhes" user "B.Adhesive")
@@
   )
   (setup
+    (stackup
+      (layer "F.SilkS" (type "Top Silk Screen"))
+      (layer "F.Paste" (type "Top Solder Paste"))
+      (layer "F.Mask" (type "Top Solder Mask") (thickness 0.01))
+      (layer "F.Cu" (type "copper") (thickness 0.035))
+      (layer "dielectric 1" (type "core") (thickness 0.48) (material "FR4") (epsilon_r 4.5) (loss_tangent 0.02))
+      (layer "In1.Cu" (type "copper") (thickness 0.035))
+      (layer "dielectric 2" (type "prepreg") (thickness 0.48) (material "FR4") (epsilon_r 4.5) (loss_tangent 0.02))
+      (layer "In2.Cu" (type "copper") (thickness 0.035))
+      (layer "dielectric 3" (type "core") (thickness 0.48) (material "FR4") (epsilon_r 4.5) (loss_tangent 0.02))
+      (layer "B.Cu" (type "copper") (thickness 0.035))
+      (layer "B.Mask" (type "Bottom Solder Mask") (thickness 0.01))
+      (layer "B.Paste" (type "Bottom Solder Paste"))
+      (layer "B.SilkS" (type "Bottom Silk Screen"))
+      (copper_finish "None")
+      (dielectric_constraints no)
+    )
     (pad_to_mask_clearance 0)
+    (solder_mask_min_width 0.1)
     (pcbplotparams
       (layerselection 0x00010fc_ffffffff)
@@
     (fp_line (start 4.555 7.94) (end 4.555 -7.81)
       (stroke (width 0.1) (type solid)) (layer "F.Fab"))
-    (pad "" np_thru_hole circle (at -57.165 2.54 180) (size 3.25 3.25) (drill 3.25) (layers "F&B.Cu" "*.Mask"))
-    (pad "" np_thru_hole circle (at 2.775 2.54 180) (size 3.25 3.25) (drill 3.25) (layers "F&B.Cu" "*.Mask"))
+    (pad "" np_thru_hole circle (at -57.165 2.54 180) (size 3.25 3.25) (drill 3.25) (layers "*.Cu" "*.Mask"))
+    (pad "" np_thru_hole circle (at 2.775 2.54 180) (size 3.25 3.25) (drill 3.25) (layers "*.Cu" "*.Mask"))
     (pad "1" thru_hole circle (at 0 0 180) (size 1.3 1.3) (drill 0.9) (layers "*.Cu" "*.Mask")
       (net 47 "Net-(J1A-BI_DA+)") (pinfunction "BI_DA+") (pintype "passive"))

Commit message: update pcb
Parts:
- C88: moved to F.Cu
- TP1, TP10, TP2, TP4, TP5, TP6, TP7, TP8, TP9: moved to B.Cu
- moved FID1 18.7 mm to (74.6, -2.54)
- moved FID4 18.7 mm to (74.6, -2.54)
- moved C47 6.25 mm to (24.1, -16.3), turned to 180 degrees
- moved C21 6.07 mm to (56.3, -2.54), turned to -90 degrees
- moved C42 5.03 mm to (55.4, -8.38), turned to -90 degrees
- moved C88 4.23 mm to (31.0, -1.52), turned to -90 degrees
- moved JP2 4.18 mm to (27.9, -9.53), turned to -90 degrees
- moved TP6 3.78 mm to (32.3, -3.81)
- moved C43 3.52 mm to (24.1, -14.6)
- moved FID3 3.37 mm to (20.1, -17.7)
- moved C71 3.20 mm to (36.8, -6.07)
- moved C84 3.20 mm to (35.8, -6.07)
- moved C59 3.20 mm to (34.8, -6.07)
- moved C48 3.05 mm to (14.7, -14.7)
- moved C38 2.93 mm to (6.10, -15.7)
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Routing:
- net +1V1: track 0.00 -> 163.0 mm, vias 0 -> 19
- net +3V3: track 0.00 -> 160.8 mm, vias 0 -> 13
- net /Y1-: track 0.00 -> 111.3 mm, vias 0 -> 8
- net GNDREF: track 0.00 -> 96.1 mm
- net /Y3+: track 0.00 -> 83.5 mm, vias 0 -> 2
- net /Y1+: track 0.00 -> 56.6 mm, vias 0 -> 2
- net +5V: track 0.00 -> 26.8 mm, vias 0 -> 2
- net Net-(D4-K): track 0.00 -> 24.9 mm, vias 0 -> 1
- net Net-(JP1-B): track 0.00 -> 22.6 mm
- net Net-(D2-A): track 0.00 -> 21.4 mm, vias 0 -> 2
- net Net-(TR2B-TD4-): track 0.00 -> 20.8 mm
- net Net-(TR1A-TD1+): track 0.00 -> 20.3 mm
- net Net-(JP2-B): track 0.00 -> 19.9 mm
- net Net-(J4-Pin_1): track 0.00 -> 19.3 mm, vias 0 -> 1
- net Net-(TR2B-TD4+): track 0.00 -> 19.0 mm
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- added copper zone on B.Cu, net GND
- added copper zone on F.Cu, net GND
- added copper zone on In1.Cu, net GND
- added copper zone on In2.Cu, net GND

Commit message: finished with tracing
Parts:
- moved D1 16.5 mm to (79.8, -24.5), turned to 0 degrees
- moved C26 15.1 mm to (78.4, -20.6), turned to 0 degrees
- moved C24 14.2 mm to (73.7, -23.0)
- moved J3 6.49 mm to (77.6, -31.2)
- moved C28 6.45 mm to (73.7, -20.6)
- moved C40 1.31 mm to (82.3, -21.0), turned to 90 degrees
- moved R28 0.55 mm to (78.0, -18.0)
- moved R29 0.46 mm to (75.3, -17.5)
- moved R25 0.40 mm to (72.8, -17.4)
Routing:
- net +5C: track 4.71 -> 101.3 mm, vias 2 -> 3
- net +24V: track 0.00 -> 15.1 mm
- net Net-(D3-K): track 0.00 -> 14.3 mm
- net Net-(D1-A): track 0.00 -> 13.4 mm
- net Net-(U4-DC): track 0.00 -> 10.1 mm
- net Net-(U4-Vfb): track 0.00 -> 4.77 mm
- net Net-(U4-TC): track 0.00 -> 3.25 mm

Commit message: update silk
Parts:
- moved FID3 43.0 mm to (63.0, -15.2)
Routing:
- net +3V3: track 160.8 -> 161.4 mm
