File: hardware/main.kicad_sch (KiCad schematic)
At the start: 204 parts, among them J1 98424-G52-06ALF, J9 TYPE-C-31-M-12, U2 MC34063AD, U5 MT3420B, Y1 SX3B25.000F1510F30

Commit message: init pcb
Parts:
- gave numbers to parts that had none: 7
- renumbered C89 to C1, C90 to C10, C91 to C11, C92 to C12, C89 to C13, C90 to C14, C91 to C15, C92 to C16, C105 to C17, C105 to C18, C105 to C19, C90 to C2, C105 to C20, C174 to C21, C174 to C22, C43 to C23, C187 to C25, C187 to C27, C91 to C3, C194 to C30, C189 to C31, C189 to C32, C191 to C33, C82 to C34, C82 to C35, C82 to C36, C191 to C37, C191 to C38, C191 to C39, C92 to C4, C85 to C41, C85 to C42, C85 to C43, C191 to C44, C87 to C45, C87 to C46, C87 to C47, C191 to C48, C191 to C49, C89 to C5, C36 to C50, C36 to C51, C38 to C52, C38 to C53, C87 to C54, C87 to C55, C87 to C56, C87 to C57, C87 to C58, C87 to C59, C90 to C6, C87 to C60, C87 to C61, C87 to C62, C87 to C63, C40 to C64, C40 to C65, C87 to C66, C87 to C67, C43 to C68, C43 to C69, C91 to C7, C87 to C70, C87 to C71, C45 to C72, C45 to C73, C87 to C74, C87 to C75, C191 to C76, C191 to C77, C87 to C78, C87 to C79, C92 to C8, C191 to C80, C191 to C81, C87 to C82, C87 to C83, C87 to C84, C87 to C85, C191 to C86, C191 to C87, C87 to C88, C87 to C89, C89 to C9, C10 to C?, C7 to C?, C9 to C?, C5 to C?, C14 to C?, D3 to D2, D4 to D?, D2 to D?, J9 to J2, J1 to J?, JP4 to JP1, JP4 to JP2, L4 to L1, L8 to L3, L8 to L4, L8 to L5, L4 to L6, L4 to L7, L1 to L?, R50 to R1, R51 to R10, R52 to R11, R53 to R12, R50 to R13, R51 to R14, R52 to R15, R53 to R16, R29 to R17, R29 to R18, R128 to R19, R51 to R2, R50 to R20, R75 to R21, R166 to R22, R167 to R23, R136 to R24, R128 to R26, R50 to R27, R52 to R3, R75 to R30, R75 to R31, R75 to R32, R75 to R33, R75 to R34, R75 to R35, R75 to R36, R75 to R37, R75 to R38, R75 to R39, R53 to R4, R75 to R40, R75 to R41, R75 to R42, R75 to R43, R75 to R44, R75 to R45, R75 to R46, R26 to R47, R26 to R48, R28 to R49, R50 to R5, R29 to R50, R28 to R51, R29 to R52, R51 to R6, R52 to R7, R53 to R8, R50 to R9, R6 to R?, R8 to R?, R7 to R?, TP2 to TP1, TP2 to TP10, TP2 to TP3, TP2 to TP4, TP2 to TP5, TP2 to TP6, TP2 to TP7, TP2 to TP8, TP2 to TP9, U5 to U6, U2 to U?

Commit message: The layout of the board
Parts:
- removed C?: 470p, Capacitor_SMD:C_0805_2012Metric, symbol Device:C_Small
- removed C? (x2): 10u, Capacitor_Tantalum_SMD:CP_EIA-7343-31_Kemet-D, symbol Device:C_Polarized_Small
- removed D?: STPS2L40U, Diode_SMD:D_SMB, symbol Device:D_Small
- removed TR1, TR2: 82FB-02NL, MAS_Package_nostd:Transformer_Ethernet_YDS-Tech_82FB-02NL, symbol MAS_Transformers:82FB-02NL
- removed unit 2 of U1
- removed unit 1 of U1
- added C29: 150p, Capacitor_SMD:C_0805_2012Metric, symbol Device:C_Small
- added C90: 10n, Capacitor_SMD:C_0402_1005Metric, symbol Device:C_Small
- added C? (x2): 2.2u, Capacitor_SMD:C_1206_3216Metric, symbol Device:C_Small
- added D4: MBR0540, Diode_SMD:D_SOD-123, symbol Diode:MBR0540
- added TR1, TR2: G5002CG, MAS_Package_nostd:Transformer_Ethernet_YDS-Tech_G5002CG, symbol MAS_Transformers:G5002CG
- C1, C10, C11, C12, C13, C14, C15, C16, C2, C23, C3, C30, C4, C5, C52, C53, C6, C68, C69, C7, C8, C9: footprint Capacitor_SMD:C_0603_1608Metric -> Capacitor_SMD:C_0402_1005Metric; Voltage 50v -> 16v; lcsc C14663 -> C1525
- C21, C22: footprint Capacitor_SMD:C_0603_1608Metric -> Capacitor_SMD:C_0402_1005Metric; lcsc C342893 -> C1557
- C45, C46, C47: footprint Capacitor_SMD:C_0603_1608Metric -> Capacitor_SMD:C_0402_1005Metric; lcsc C1588 -> C1523
- C54, C55, C56, C57, C58, C59, C60, C61, C62, C63, C66, C67, C70, C71, C74, C75, C78, C79, C82, C83, C84, C85, C88, C89: footprint Capacitor_SMD:C_0603_1608Metric -> Capacitor_SMD:C_0402_1005Metric; lcsc C57112 -> C15195
- D2: lcsc (none) -> C116159
- JP1, JP2: value J_Boot -> jump
- R1, R10, R11, R12, R13, R14, R15, R16, R2, R3, R4, R5, R6, R7, R8, R9: footprint Resistor_SMD:R_0603_1608Metric -> Resistor_SMD:R_0402_1005Metric; lcsc C4275 -> C25133
- R17, R18, R52: footprint Resistor_SMD:R_0603_1608Metric -> Resistor_SMD:R_0402_1005Metric; lcsc C31850 -> C25768
- R19: footprint Resistor_SMD:R_0603_1608Metric -> Resistor_SMD:R_0402_1005Metric; lcsc C227773 -> C145071
- R21, R22, R23, R30, R31, R32, R33, R34, R35, R36, R37, R38, R39, R40, R41, R42, R43, R44, R45, R46: footprint Resistor_SMD:R_0603_1608Metric -> Resistor_SMD:R_0402_1005Metric; lcsc C23162 -> C25900
- R24: footprint Resistor_SMD:R_0603_1608Metric -> Resistor_SMD:R_0402_1005Metric
- R26, R47, R48, R49, R51: footprint Resistor_SMD:R_0603_1608Metric -> Resistor_SMD:R_0402_1005Metric; lcsc C25803 -> C25741
- TP1, TP10, TP2, TP3, TP4, TP5, TP6, TP7, TP8, TP9: footprint TestPoint:TestPoint_Pad_D1.0mm -> MAS_Package_std:TestPoint_Pad_D0.5mm
- U1: lcsc (none) -> C2803243
Connections:
- net +1V1: now also C90.1
- net +24V: now also C?.1, C?.1
- net GND: now also C29.2, C90.2, C?.2, C?.2
- net at R13.2: now also TR2.27 (CMT4)
- net at R7.2: now also TR1.33 (CMT2)
- net at C2.2: now also TR1.8 (TCT3)
- net at C12.2: now also TR2.2 (TCT1)
- net at C5.2: now also TR1.24 (TCT4)
- net at C6.2: now also TR1.21 (TCT3)
- net at C7.2: now also TR1.18 (TCT2)
- net at C8.2: now also TR1.15 (TCT1)
- net at J1.14 (BI_DA+): now also TR1.35 (MX1+)
- net at J1.15 (BI_DA-): now also TR1.37 (MX1-)
- net at R8.2: now also TR1.36 (CMT1)
- net at J1.17 (BI_DC+): now also TR1.34 (MX2+)
- net at J1.18 (BI_DC-): now also TR1.32 (MX2-)
- net at J1.16 (BI_DB+): now also TR1.29 (MX3+)
- net at J1.19 (BI_DB-): now also TR1.31 (MX3-)
- net at R6.2: now also TR1.30 (CMT3)
- net at J1.20 (BI_DD+): now also TR1.28 (MX4+)
- net at J1.21 (BI_DD-): now also TR1.26 (MX4-)
- net at R5.2: now also TR1.27 (CMT4)
- net at C10.2: now also TR2.8 (TCT3)
- net at C16.2: now also TR2.15 (TCT1)
- net at C9.2: now also TR2.11 (TCT4)
- net at U1.3 (P2MDIDP): now also TR2.16 (TD1-)
- net at U1.4 (P2MDIDN): now also TR2.14 (TD1+)
- net at U1.124 (P2MDIAP): now also TR2.25 (TD4-)
- net at U1.125 (P2MDIAN): now also TR2.23 (TD4+)
- net at J1.27 (BI_DA+): now also TR2.48 (MX1+)
- net at J1.28 (BI_DA-): now also TR2.50 (MX1-)
- net at R12.2: now also TR2.49 (CMT1)
- net at J1.30 (BI_DC+): now also TR2.47 (MX2+)
- net at J1.31 (BI_DC-): now also TR2.45 (MX2-)
- net at R11.2: now also TR2.46 (CMT2)
- net at J1.29 (BI_DB+): now also TR2.42 (MX3+)
- net at J1.32 (BI_DB-): now also TR2.44 (MX3-)
- net at R10.2: now also TR2.43 (CMT3)
- net at J1.33 (BI_DD+): now also TR2.41 (MX4+)
- net at J1.34 (BI_DD-): now also TR2.39 (MX4-)
- net at R9.2: now also TR2.40 (CMT4)
- net at U1.126 (P2MDIBP): now also TR2.22 (TD3-)
- net at U1.127 (P2MDIBN): now also TR2.20 (TD3+)
- net at C11.2: now also TR2.5 (TCT2)
- net at U1.1 (P2MDICP): now also TR2.19 (TD2-)
- net at U1.2 (P2MDICN): now also TR2.17 (TD2+)
- net at C14.2: now also TR2.21 (TCT3)
- net at C37.1, C39.1, C44.1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: now also D4.1 (K)
- net at C13.2: now also TR2.24 (TCT4)
- net at U1.6 (P3MDIAP): now also TR2.12 (TD4-)
- net at U1.7 (P3MDIAN): now also TR2.10 (TD4+)
- net at U1.8 (P3MDIBP): now also TR2.9 (TD3-)
- net at U1.9 (P3MDIBN): now also TR2.7 (TD3+)
- net at C15.2: now also TR2.18 (TCT2)
- net at U1.11 (P3MDICP): now also TR2.6 (TD2-)
- net at U1.12 (P3MDICN): now also TR2.4 (TD2+)
- net at U1.13 (P3MDIDP): now also TR2.3 (TD1-)
- net at U1.14 (P3MDIDN): now also TR2.1 (TD1+)
- net at J1.40 (BI_DA+): now also TR2.35 (MX1+)
- net at J1.41 (BI_DA-): now also TR2.37 (MX1-)
- net at R16.2: now also TR2.36 (CMT1)
- net at J1.43 (BI_DC+): now also TR2.34 (MX2+)
- net at J1.44 (BI_DC-): now also TR2.32 (MX2-)
- net at R15.2: now also TR2.33 (CMT2)
- net at J1.42 (BI_DB+): now also TR2.29 (MX3+)
- net at J1.45 (BI_DB-): now also TR2.31 (MX3-)
- net at R14.2: now also TR2.30 (CMT3)
- net at J1.46 (BI_DD+): now also TR2.28 (MX4+)
- net at J1.47 (BI_DD-): now also TR2.26 (MX4-)
- net at R4.2: now also TR1.49 (CMT1)
- net at C32.1, F1.1, L1.2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: now also D4.2 (A)
- net at C3.2: now also TR1.5 (TCT2)
- net at C4.2: now also TR1.2 (TCT1)
- net at R3.2: now also TR1.46 (CMT2)
- net at U?.3 (TC): now also C29.1
- net at U1.25 (P4MDIAP): now also TR1.25 (TD4-)
- net at U1.26 (P4MDIAN): now also TR1.23 (TD4+)
- net at U1.27 (P4MDIBP): now also TR1.22 (TD3-)
- net at U1.28 (P4MDIBN): now also TR1.20 (TD3+)
- net at U1.30 (P4MDICP): now also TR1.19 (TD2-)
- net at U1.31 (P4MDICN): now also TR1.17 (TD2+)
- net at U1.32 (P4MDIDP): now also TR1.16 (TD1-)
- net at U1.33 (P4MDIDN): now also TR1.14 (TD1+)
- net at R1.2: now also TR1.40 (CMT4)
- net at U1.35 (P5MDIAP): now also TR1.12 (TD4-)
- net at U1.36 (P5MDIAN): now also TR1.10 (TD4+)
- net at U1.37 (P5MDIBP): now also TR1.9 (TD3-)
- net at U1.38 (P5MDIBN): now also TR1.7 (TD3+)
- net at U1.40 (P5MDICP): now also TR1.6 (TD2-)
- net at U1.41 (P5MDICN): now also TR1.4 (TD2+)
- net at U1.42 (P5MDIDP): now also TR1.3 (TD1-)
- net at U1.43 (P5MDIDN): now also TR1.1 (TD1+)
- net at C1.2: now also TR1.11 (TCT4)
- net at J1.1 (BI_DA+): now also TR1.48 (MX1+)
- net at J1.2 (BI_DA-): now also TR1.50 (MX1-)
- net at J1.3 (BI_DB+): now also TR1.42 (MX3+)
- net at J1.4 (BI_DC+): now also TR1.47 (MX2+)
- net at J1.5 (BI_DC-): now also TR1.45 (MX2-)
- net at J1.6 (BI_DB-): now also TR1.44 (MX3-)
- net at J1.7 (BI_DD+): now also TR1.41 (MX4+)
- net at J1.8 (BI_DD-): now also TR1.39 (MX4-)
- net at R2.2: now also TR1.43 (CMT3)
- no-connect marks 32 -> 16
Other:
- moved on the sheet: U1E, U1F

Commit message: update sch and pcb
Parts:
- removed BT1: BH-18650-B1BA002, MAS_Package_nostd:BatteryHolder_BH-18650-B1BA002, symbol Device:Battery_Cell
- removed D?: STPS2L40U, Diode_SMD:D_SMB, symbol Device:D_Small
- added D?: SS14, Diode_SMD:D_SMA, symbol Device:D_Small
- added J4: batt, Connector_PinHeader_2.54mm:PinHeader_1x02_P2.54mm_Vertical, symbol Connector:Conn_01x02_Male
- C29: footprint Capacitor_SMD:C_0805_2012Metric -> Capacitor_SMD:C_0603_1608Metric; lcsc C1716 -> C1594
- D?: value STPS2L40U -> SS14; footprint Diode_SMD:D_SMB -> Diode_SMD:D_SMA; chipdip 2666823191 -> (none); lcsc C169095 -> C2480; promelec 126735 -> (none)
- R?: value 0.33R -> 0.5R; footprint Resistor_SMD:R_1206_3216Metric -> Resistor_SMD:R_0805_2012Metric; lcsc C25337 -> C912543; promelec 54682 -> (none)
- R?: footprint Resistor_SMD:R_0805_2012Metric -> Resistor_SMD:R_0603_1608Metric; chipdip 9000079488 -> (none); lcsc C17379 -> C22765
- R?: footprint Resistor_SMD:R_0805_2012Metric -> Resistor_SMD:R_0603_1608Metric; chipdip 9000079499 -> (none); lcsc C18359 -> C22980
Connections:
- net +24V: now also D?.1 (K)
- net GND: now also J4.2 (Pin_2)
- net at J?.1 (Pin_1), J?.2 (Pin_2), J?.3 (Pin_3): now also D?.2 (A)
- net at F1.2: now also J4.1 (Pin_1)
Changed lines of the file:
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@@
     (stroke (width 0) (type default))
   )
-  (wire (pts (xy 323.85 321.31) (xy 323.85 325.12))
+  (wire (pts (xy 322.58 321.31) (xy 322.58 327.66))
     (stroke (width 0) (type default))
   )
@@
     (stroke (width 0) (type default))
   )
-  (wire (pts (xy 321.31 321.31) (xy 323.85 321.31))
+  (wire (pts (xy 321.31 321.31) (xy 322.58 321.31))
     (stroke (width 0) (type default))
   )
@@
     (stroke (width 0) (type default))
   )
+  (wire (pts (xy 322.58 330.2) (xy 323.85 330.2))
+    (stroke (width 0) (type default))
+  )
   (wire (pts (xy 510.54 330.2) (xy 510.54 331.47))
     (stroke (width 0) (type default))
@@
     (stroke (width 0) (type default))
   )
+  (wire (pts (xy 322.58 327.66) (xy 323.85 327.66))
+    (stroke (width 0) (type default))
+  )
   (wire (pts (xy 515.62 154.94) (xy 513.08 154.94))
     (stroke (width 0) (type default))
@@
     (stroke (width 0) (type default))
   )
-  (wire (pts (xy 314.96 336.55) (xy 323.85 336.55))
+  (wire (pts (xy 314.96 336.55) (xy 322.58 336.55))
     (stroke (width 0) (type default))
   )
@@
     (stroke (width 0) (type default))
   )
-  (wire (pts (xy 323.85 332.74) (xy 323.85 336.55))
+  (wire (pts (xy 322.58 330.2) (xy 322.58 336.55))
     (stroke (width 0) (type default))
   )
@@
       (effects (font (size 1.27 1.27)))
     )
-    (property "Value" "STPS2L40U" (at 294.64 287.02 0)
+    (property "Value" "SS14" (at 294.64 287.02 0)
       (effects (font (size 1.27 1.27)))
     )
-    (property "Footprint" "Diode_SMD:D_SMB" (at 297.18 287.02 90)
+    (property "Footprint" "Diode_SMD:D_SMA" (at 297.18 287.02 90)
       (effects (font (size 1.27 1.27)) hide)
     )
@@
       (effects (font (size 1.27 1.27)) hide)
     )
-    (property "chipdip" "2666823191" (at 297.18 287.02 0)
-      (effects (font (size 1.27 1.27)) hide)
-    )
-    (property "lcsc" "C169095" (at 297.18 287.02 0)
-      (effects (font (size 1.27 1.27)) hide)
-    )
-    (property "promelec" "126735" (at 297.18 287.02 0)
+    (property "lcsc" "C2480" (at 297.18 287.02 0)
       (effects (font (size 1.27 1.27)) hide)
     )
@@
     )
   )
-  (symbol (lib_id "Device:D_Small") (at 232.41 271.78 0) (mirror y) (unit 1)
-    (in_bom yes) (on_board yes) (dnp no)
-    (property "Reference" "D?" (at 232.41 266.573 0)
-      (effects (font (size 1.27 1.27)))
-    )
-    (property "Value" "STPS2L40U" (at 232.41 269.24 0)
-      (effects (font (size 1.27 1.27)))
-    )
-    (property "Footprint" "Diode_SMD:D_SMB" (at 232.41 271.78 90)
-      (effects (font (size 1.27 1.27)) hide)
-    )
-    (property "Datasheet" "~" (at 232.41 271.78 90)
-      (effects (font (size 1.27 1.27)) hide)
-    )
-    (property "chipdip" "2666823191" (at 232.41 271.78 0)
-      (effects (font (size 1.27 1.27)) hide)
-    )
-    (property "lcsc" "C169095" (at 232.41 271.78 0)
-      (effects (font (size 1.27 1.27)) hide)
-    )
-    (property "promelec" "126735" (at 232.41 271.78 0)
-      (effects (font (size 1.27 1.27)) hide)
-    )
-    (pin "1")
-    (pin "2")
-    (instances
-      (project "main"
-        (path "/156d6217-48e9-4298-9a4f-ae9337ac0371"
-          (reference "D?") (unit 1)
-        )
-      )
-      (project "main"
-        (path "/c6e5d5ba-43a3-4ff8-a766-3efdb024d1f4"
-          (reference "D1") (unit 1)
-        )
-      )
-    )
-  )
   (symbol (lib_id "Device:C_Small") (at 240.03 180.34 90) (unit 1)
     (in_bom yes) (on_board yes) (dnp no)
@@
       (effects (font (size 1.27 1.27)) (justify right))
     )
-    (property "Value" "0.33R" (at 294.8686 266.573 0)
+    (property "Value" "0.5R" (at 294.8686 266.573 0)
       (effects (font (size 1.27 1.27)) (justify right))
     )
-    (property "Footprint" "Resistor_SMD:R_1206_3216Metric" (at 293.37 265.43 0)
+    (property "Footprint" "Resistor_SMD:R_0805_2012Metric" (at 293.37 265.43 0)
       (effects (font (size 1.27 1.27)) hide)
     )
@@
       (effects (font (size 1.27 1.27)) hide)
     )
-    (property "promelec" "54682" (at 293.37 265.43 0)
-      (effects (font (size 1.27 1.27)) hide)
-    )
-    (property "lcsc" "C25337" (at 293.37 265.43 0)
+    (property "lcsc" "C912543" (at 293.37 265.43 0)
       (effects (font (size 1.27 1.27)) hide)
     )
@@
       (effects (font (size 1.27 1.27)) (justify right))
     )
-    (property "Footprint" "Resistor_SMD:R_0805_2012Metric" (at 314.96 293.37 0)
+    (property "Footprint" "Resistor_SMD:R_0603_1608Metric" (at 314.96 293.37 0)
       (effects (font (size 1.27 1.27)) hide)
     )
@@
       (effects (font (size 1.27 1.27)) hide)
     )
-    (property "chipdip" "9000079488" (at 314.96 293.37 0)
-      (effects (font (size 1.27 1.27)) hide)
-    )
-    (property "lcsc" "C17379" (at 314.96 293.37 0)
+    (property "lcsc" "C22765" (at 314.96 293.37 0)
       (effects (font (size 1.27 1.27)) hide)
     )
@@
     )
   )
-  (symbol (lib_id "Device:Battery_Cell") (at 323.85 330.2 0) (unit 1)
-    (in_bom yes) (on_board yes) (dnp no)
-    (property "Reference" "BT1" (at 326.39 326.39 0)
-      (effects (font (size 1.27 1.27)) (justify left))
-    )
-    (property "Value" "BH-18650-B1BA002" (at 327.66 329.4379 0)
-      (effects (font (size 1.27 1.27)) (justify left) hide)
-    )
-    (property "Footprint" "MAS_Package_nostd:BatteryHolder_BH-18650-B1BA002" (at 323.85 328.676 90)
-      (effects (font (size 1.27 1.27)) hide)
-    )
-    (property "Datasheet" "https://datasheet.lcsc.com/lcsc/2204021730_MYOUNG-BH-18650-B1BA002_C2988620.pdf" (at 323.85 328.676 90)
-      (effects (font (size 1.27 1.27)) hide)
-    )
-    (property "lcsc" "C2988620" (at 323.85 330.2 0)
-      (effects (font (size 1.27 1.27)) hide)
-    )
-    (pin "1")
-    (pin "2")
-    (instances
-      (project "main"
-        (path "/c6e5d5ba-43a3-4ff8-a766-3efdb024d1f4"
-          (reference "BT1") (unit 1)
-        )
-      )
-    )
-  )
   (symbol (lib_id "Device:C_Small") (at 448.31 190.5 0) (unit 1)
     (in_bom yes) (on_board yes) (dnp no)
@@
       (effects (font (size 1.27 1.27)) (justify left))
     )
-    (property "Footprint" "Capacitor_SMD:C_0805_2012Metric" (at 266.7 285.75 0)
+    (property "Footprint" "Capacitor_SMD:C_0603_1608Metric" (at 266.7 285.75 0)
       (effects (font (size 1.27 1.27)) hide)
     )
@@
       (effects (font (size 1.27 1.27)) hide)
     )
-    (property "lcsc" "C1716" (at 266.7 285.75 0)
+    (property "lcsc" "C1594" (at 266.7 285.75 0)
       (effects (font (size 1.27 1.27)) hide)
     )
@@
     )
   )
+  (symbol (lib_id "Connector:Conn_01x02_Male") (at 328.93 327.66 0) (mirror y) (unit 1)
+    (in_bom yes) (on_board yes) (dnp no)
+    (property "Reference" "J4" (at 330.2 329.565 0)
+      (effects (font (size 1.27 1.27)) (justify right))
+    )
+    (property "Value" "batt" (at 330.2 327.025 0)
+      (effects (font (size 1.27 1.27)) (justify right))
+    )
+    (property "Footprint" "Connector_PinHeader_2.54mm:PinHeader_1x02_P2.54mm_Vertical" (at 328.93 327.66 0)
+      (effects (font (size 1.27 1.27)) hide)
+    )
+    (property "Datasheet" "~" (at 328.93 327.66 0)
+      (effects (font (size 1.27 1.27)) hide)
+    )
+    (property "lcsc" "C492401" (at 328.93 327.66 0)
+      (effects (font (size 1.27 1.27)) hide)
+    )
+    (pin "1")
+    (pin "2")
+    (instances
+      (project "main"
+        (path "/156d6217-48e9-4298-9a4f-ae9337ac0371"
+          (reference "J4") (unit 1)
+        )
+      )
+      (project "main"
+        (path "/c6e5d5ba-43a3-4ff8-a766-3efdb024d1f4"
+          (reference "J4") (unit 1)
+        )
+      )
+    )
+  )
   (symbol (lib_id "Device:C_Small") (at 393.7 337.82 0) (unit 1)
     (in_bom yes) (on_board yes) (dnp no)
@@
     )
   )
+  (symbol (lib_id "Device:D_Small") (at 232.41 271.78 0) (mirror y) (unit 1)
+    (in_bom yes) (on_board yes) (dnp no)
+    (property "Reference" "D?" (at 232.41 266.573 0)
+      (effects (font (size 1.27 1.27)))
+    )
+    (property "Value" "SS14" (at 232.41 269.24 0)
+      (effects (font (size 1.27 1.27)))
+    )
+    (property "Footprint" "Diode_SMD:D_SMA" (at 232.41 271.78 90)
+      (effects (font (size 1.27 1.27)) hide)
+    )
+    (property "Datasheet" "~" (at 232.41 271.78 90)
+      (effects (font (size 1.27 1.27)) hide)
+    )
+    (property "lcsc" "C2480" (at 232.41 271.78 0)
+      (effects (font (size 1.27 1.27)) hide)
+    )
+    (pin "1")
+    (pin "2")
+    (instances
+      (project "main"
+        (path "/156d6217-48e9-4298-9a4f-ae9337ac0371"
+          (reference "D?") (unit 1)
+        )
+      )
+      (project "main"
+        (path "/c6e5d5ba-43a3-4ff8-a766-3efdb024d1f4"
+          (reference "D1") (unit 1)
+        )
+      )
+    )
+  )
   (symbol (lib_id "Device:R_Small") (at 340.36 120.65 270) (mirror x) (unit 1)
     (in_bom yes) (on_board yes) (dnp no)
@@
       (effects (font (size 1.27 1.27)) (justify right))
     )
-    (property "Footprint" "Resistor_SMD:R_0805_2012Metric" (at 314.96 285.75 0)
+    (property "Footprint" "Resistor_SMD:R_0603_1608Metric" (at 314.96 285.75 0)
       (effects (font (size 1.27 1.27)) hide)
     )
@@
       (effects (font (size 1.27 1.27)) hide)
     )
-    (property "chipdip" "9000079499" (at 314.96 285.75 0)
-      (effects (font (size 1.27 1.27)) hide)
-    )
-    (property "lcsc" "C18359" (at 314.96 285.75 0)
+    (property "lcsc" "C22980" (at 314.96 285.75 0)
       (effects (font (size 1.27 1.27)) hide)
     )

Commit message: fix pcb and check drc
Parts:
- added R53, R54, R55: 470R, Resistor_SMD:R_0402_1005Metric, symbol Device:R_Small
- added TP11: TestPoint, MAS_Package_std:TestPoint_Pad_D0.5mm, symbol Connector:TestPoint
- added unit 1 of U1
- added unit 2 of U1
- R32: value 4.7k -> 470R; lcsc C25900 -> C25117
Connections:
- net +3V3: now also R53.2, R54.2, R55.2
- net G1+: now also R55.1
- net G1-: now also U1.74 (P5LED0), TP11.1
- net G2+: now also R54.1
- net G2-: now also R34.1, U1.80 (P4LED0/SLED_P6B/STRP_EEPROM_MOD)
- net G3+: now also R53.1
- net G3-: now also R37.1, U1.84 (P3LED0/SLED_P2B/STRP_EN_FLASH)
- net G4+: now also R32.1
- net G4-: now also R39.1, U1.86 (P2LED0/SLED_P0B/STRP_DISAUTOLOAD)
Other:
- moved on the sheet: R30, R31, R33, R34, R35, R36, R37, R38, R39, R40, R41, R42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

Commit message: fix wire
Parts:
- J1: lcsc C86578 -> C138390
Changed lines of the file:
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@@
       (effects (font (size 1.27 1.27) italic) hide)
     )
-    (property "lcsc" "C86578" (at 147.32 265.43 0)
+    (property "lcsc" "C138390" (at 147.32 265.43 0)
       (effects (font (size 1.27 1.27) italic) hide)
     )
@@
       (effects (font (size 1.27 1.27) italic) hide)
     )
-    (property "lcsc" "C86578" (at 147.32 180.34 0)
+    (property "lcsc" "C138390" (at 147.32 180.34 0)
       (effects (font (size 1.27 1.27) italic) hide)
     )
@@
       (effects (font (size 1.27 1.27) italic) hide)
     )
-    (property "lcsc" "C86578" (at 147.32 92.71 0)
+    (property "lcsc" "C138390" (at 147.32 92.71 0)
       (effects (font (size 1.27 1.27) italic) hide)
     )
@@
       (effects (font (size 1.27 1.27) italic) hide)
     )
-    (property "lcsc" "C86578" (at 147.32 353.06 0)
+    (property "lcsc" "C138390" (at 147.32 353.06 0)
       (effects (font (size 1.27 1.27) italic) hide)
     )
